File: pcb.kicad_pcb (KiCad board)
At the start: 2 copper layers, 120.7 x 70.6 mm, 12 parts, among them U1 Pico

Commit message: Final touches for Rev 1
Other:
- board text added: "5V"
- board text added: "DIN"
- board text added: "GND"
- board text added: "WS2812B (10 LEDs)"
Changed lines of the file:
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@@
     (pad_to_mask_clearance 0)
     (pcbplotparams
-      (layerselection 0x00010fc_ffffffff)
+      (layerselection 0x00010f0_ffffffff)
       (disableapertmacros false)
-      (usegerberextensions false)
+      (usegerberextensions true)
       (usegerberattributes true)
       (usegerberadvancedattributes true)
-      (creategerberjobfile true)
+      (creategerberjobfile false)
       (svguseinch false)
       (svgprecision 6)
@@
       (plotinvisibletext false)
       (sketchpadsonfab false)
-      (subtractmaskfromsilk false)
+      (subtractmaskfromsilk true)
       (outputformat 1)
       (mirror false)
-      (drillshape 1)
+      (drillshape 0)
       (scaleselection 1)
       (outputdirectory "")
@@
     (effects (font (size 1 1) (thickness 0.15)) (justify mirror))
   )
+  (gr_text "WS2812B\n(10 LEDs)" (at 92.075 89.662) (layer "B.SilkS")
+    (effects (font (size 1 1) (thickness 0.15)) (justify mirror))
+  )
   (gr_text "P2 CN" (at 173.0375 103.1875) (layer "B.SilkS")
     (effects (font (size 2 2) (thickness 0.15)) (justify mirror))
@@
     (effects (font (size 2 2) (thickness 0.15)) (justify mirror))
   )
+  (gr_text "DIN\n" (at 91.821 97.536) (layer "B.SilkS")
+    (effects (font (size 1 1) (thickness 0.15)) (justify mirror))
+  )
   (gr_text "P1 UR" (at 130.175 84.1375) (layer "B.SilkS")
     (effects (font (size 2 2) (thickness 0.15)) (justify mirror))
@@
     (effects (font (size 2 2) (thickness 0.15)) (justify mirror))
   )
+  (gr_text "5V" (at 89.408 92.964) (layer "B.SilkS")
+    (effects (font (size 1 1) (thickness 0.15)) (justify mirror))
+  )
   (gr_text "- +" (at 153.9875 79.375) (layer "B.SilkS")
     (effects (font (size 1 1) (thickness 0.15)) (justify mirror))
@@
     (effects (font (size 2 2) (thickness 0.15)) (justify mirror))
   )
+  (gr_text "GND" (at 94.488 92.964) (layer "B.SilkS")
+    (effects (font (size 1 1) (thickness 0.15)) (justify mirror))
+  )
   (gr_text "HandPump PCB Rev. 1\nhttps://github.com/dj505/handpump" (at 200.81875 125.4125) (layer "B.Mask")
