File: pcb.kicad_pcb (KiCad board)
At the start: 2 copper layers, 120.7 x 70.6 mm, 12 parts, among them U1 Pico

Commit message: ooooo fancy pcb art (+ silkscreen adjustments)
Parts:
- added G***: LOGO, LogoFootprints:Arrow_19_05mm, F.Cu at (153.9, 114.3)
- added G***: LOGO, LogoFootprints:Arrow_19_05mm, F.Cu at (192.0, 76.2)
- added G***: LOGO, LogoFootprints:Arrow_6, B.Cu at (198.1, 125.7)
- added G***: LOGO, LogoFootprints:CenterStep, F.Cu at (173.0, 95.2)
- added G***: LOGO, LogoFootprints:Arrow_19_05mm, F.Cu at (192.0, 114.3)
- added G***: LOGO, LogoFootprints:Arrow_19_05mm, F.Cu at (130.0, 76.2)
- added G***: LOGO, LogoFootprints:Arrow_19_05mm, F.Cu at (91.9, 114.3)
- added G***: LOGO, LogoFootprints:Arrow_19_05mm, F.Cu at (153.9, 76.2)
- added G***: LOGO, LogoFootprints:Arrow_19_05mm, F.Cu at (91.9, 76.2)
- added G***: LOGO, LogoFootprints:CenterStep, F.Cu at (111.0, 95.2)
- added G***: LOGO, LogoFootprints:Arrow_19_05mm, F.Cu at (130.3, 114.3)
Other:
- board text added: "HandPump PCB Rev. 2 https://github.com/dj505/handpump"
- board text removed: "HandPump PCB Rev. 1 https://github.com/dj505/handpump"

Commit message: More PCB art, some tweaking
Parts:
- added G***: LOGO, LogoFootprints:InfinitesimalLoop_18mm, B.Cu at (111.0, 114.0)
- added G***: LOGO, LogoFootprints:InfinitesimalLogo_18mm, B.Cu at (111.0, 120.7)
Other:
- board text added: "Try"
- board text added: "https://github.com/dj505/Infinitesimal"

Commit message: Clean up schematic, PCB adjustments
Connections:
- U1 pad 33: GND -> unconnected-(U1-Pad33)
- U1 pad 36: +3.3V -> unconnected-(U1-Pad36)

Commit message: add test/service buttons (oops)
Parts:
- added SW1: SW_Push, Button_Switch_THT:SW_PUSH_6mm, F.Cu at (192.0, 88.7)
- added SW2: SW_Push, Button_Switch_THT:SW_PUSH_6mm, F.Cu at (192.0, 97.3)
Connections:
- U1 pad 19: unconnected-(U1-Pad19) -> SERVICE
- U1 pad 20: unconnected-(U1-Pad20) -> TEST
Routing:
- net SERVICE: track 0.00 -> 31.5 mm
- net TEST: track 0.00 -> 24.8 mm
Other:
- board text added: "SERVICE"
- board text added: "TEST"

Commit message: actually add test/service buttons (double oops)
position not final
Other:
- board text added: "GP14"
- board text added: "GP15"
Changed lines of the file:
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@@
     (effects (font (size 1 1) (thickness 0.15)) (justify mirror))
+  )
+  (gr_text "GP15" (at 186.328 109.728 -225) (layer "B.SilkS")
+    (effects (font (size 0.8 0.8) (thickness 0.15)) (justify mirror))
   )
   (gr_text "- +" (at 130.175 79.375) (layer "B.SilkS")
@@
     (effects (font (size 1 1) (thickness 0.15)) (justify mirror))
   )
+  (gr_text "GP14" (at 186.182 107.188 -225) (layer "B.SilkS")
+    (effects (font (size 0.8 0.8) (thickness 0.15)) (justify mirror))
+  )
   (gr_text "WS2812B\n(10 LEDs)" (at 92.075 89.662) (layer "B.SilkS")
